Commit message: Aggiunto blocco ros2_control per migrazione Humble

File: helene_ros/src/hw_description/urdf/helene_hw.urdf (robot description, URDF)
Before this commit: robot helene, 9 links, 8 joints
Links:
- removed link axis_0
- removed link axis_1
- removed link axis_2
- removed link axis_3
- removed link axis_4
- removed link axis_5
- removed link axis_6
Joints:
- removed joint q2
- removed joint q3
- removed joint q4
- removed joint q5
- removed joint q6
- removed joint q7
